File: hardware/RAMs/feRAM_32k.kicad_sch (KiCad schematic)
At the start: 0 parts

Commit message: Added feRAM
Parts:
- added M?: ~, Package_SO:SOIC-28W_7.5x17.9mm_P1.27mm, symbol AGB_common:FM28V020
Connections:
- new net +3.3V: M?.28 (VCC)
- new net A0: M?.10 (A0)
- new net A1: M?.9 (A1)
- new net A10: M?.21 (A10)
- new net A11: M?.23 (A11)
- new net A12: M?.2 (A12)
- new net A13: M?.26 (A13)
- new net A14: M?.1 (A14)
- new net A2: M?.8 (A2)
- new net A3: M?.7 (A3)
- new net A4: M?.6 (A4)
- new net A5: M?.5 (A5)
- new net A6: M?.4 (A6)
- new net A7: M?.3 (A7)
- new net A8: M?.25 (A8)
- new net A9: M?.24 (A9)
- new net CS2: M?.20 (~{CS})
- new net D0: M?.11 (Q0)
- new net D1: M?.12 (Q1)
- new net D2: M?.13 (Q2)
- new net D3: M?.15 (Q3)
- new net D4: M?.16 (Q4)
- new net D5: M?.17 (Q5)
- new net D6: M?.18 (Q6)
- new net D7: M?.19 (Q7)
- new net GND: M?.14 (GND)
- new net R: M?.22 (~{OE})
- new net W: M?.27 (~{WE})
- no-connect marks 0 -> 1
